Commit message: Set correct joint limits for simulation

File: src/pkg_gripper/urdf/robotiq_arg2f_85_model_macro.xacro (robot description, xacro)
@@ -146,5 +146,5 @@
       <child link="${prefix}${fingerprefix}_inner_finger" />
       <axis xyz="1 0 0" />
-      <limit lower="0" upper="0.8757" velocity="2.0" effort="1000" />
+      <limit lower="-3.14" upper="3.14" velocity="2.0" effort="1000" />
       <mimic joint="${prefix}finger_joint" multiplier="-1" offset="0" />
     </joint>

File: src/pkg_robot_gripper/urdf/ur5_robotiq.xacro (robot description, xacro)
@@ -4,8 +4,9 @@
     <xacro:include filename="$(find ur_description)/urdf/ur5.xacro" />
     <!-- Include Robotiq 2F-85 xacro -->
-    <xacro:include filename="$(find robotiq_2f_85_gripper_visualization)/urdf/robotiq_arg2f_85_model.xacro" />
-    <joint name="wrist_to_gripper" type="fixed">
+    <xacro:include filename="$(find pkg_gripper)/urdf/robotiq_arg2f_85_model_macro.xacro" />
+    <xacro:robotiq_arg2f_85 prefix=""/>
+    <joint name="tool_to_gripper" type="fixed">
         <origin xyz="0 0 0" rpy="0 0 0"/>
-        <parent link="wrist_3_link"/>  <!-- UR5的末端链接 -->
+        <parent link="tool0"/>  <!-- UR5的末端链接 -->
         <child link="robotiq_arg2f_base_link"/>  <!-- Robotiq的根链接 -->
     </joint>
