Commit message: Add controllers

File: src/pkg_gripper/urdf/robotiq_85_gripper.transmission.xacro (robot description, xacro)
@@ -5,11 +5,8 @@
       <type>transmission_interface/SimpleTransmission</type>
       <joint name="${prefix}robotiq_85_left_knuckle_joint">
-        <hardwareInterface>PositionJointInterface</hardwareInterface>
-        <!-- <hardwareInterface>EffortJointInterface</hardwareInterface> -->
+        <hardwareInterface>hardware_interface/EffortJointInterface</hardwareInterface>
       </joint>
       <actuator name="${prefix}robotiq_85_left_knuckle_motor">
         <mechanicalReduction>1</mechanicalReduction>
-        <hardwareInterface>PositionJointInterface</hardwareInterface>
-        <!-- <hardwareInterface>EfforJointInterface</hardwareInterface> -->
       </actuator>
     </transmission>

File: src/pkg_gripper/urdf/robotiq_description.xacro (robot description, xacro)
@@ -5,5 +5,10 @@
     <xacro:include filename="$(find pkg_gripper)/urdf/robotiq_85_gripper.urdf.xacro" />
     <xacro:robotiq_85_gripper prefix="" parent="world" >
-    <origin xyz="0 0 0.004" rpy="0 ${-pi/2} ${pi}"/>
+    <origin xyz="0 0 0.004" rpy="0 ${-pi/2} ${pi}"/>>>
     </xacro:robotiq_85_gripper>
+    <gazebo>
+        <plugin name="gazebo_ros_control" filename="libgazebo_ros_control.so">
+            <robotNamespace>/</robotNamespace>
+        </plugin>
+    </gazebo>
 </robot>
