Commit message: Fix joint limits issues

File: src/pkg_gripper/urdf/robotiq_85_gripper.urdf.xacro (robot description, xacro)
@@ -34,10 +34,10 @@
       <limit lower="0.0" upper="0.80285" velocity="0.5" effort="1000"/>
     </joint>
-    <joint name="${prefix}robotiq_85_right_knuckle_joint" type="continuous">
+    <joint name="${prefix}robotiq_85_right_knuckle_joint" type="revolute">
       <parent link="${prefix}robotiq_85_base_link"/>
       <child link="${prefix}robotiq_85_right_knuckle_link"/>
       <axis xyz="0 0 1"/>
       <origin rpy="0.0 0.0 0.0" xyz="0.05490451627 -0.03060114443 0.0"/>
-      <limit lower="-3.14" upper="3.14" velocity="100.0" effort="1000"/>
+      <limit lower="0" upper="0.80285" velocity="100.0" effort="1000"/>
       <mimic joint="${prefix}robotiq_85_left_knuckle_joint"/>
     </joint>
@@ -128,18 +128,18 @@
       </inertial>
     </link>
-    <joint name="${prefix}robotiq_85_left_inner_knuckle_joint" type="continuous">
+    <joint name="${prefix}robotiq_85_left_inner_knuckle_joint" type="revolute">
       <parent link="${prefix}robotiq_85_base_link"/>
       <child link="${prefix}robotiq_85_left_inner_knuckle_link"/>
       <axis xyz="0 0 1"/>
       <origin xyz="0.06142 0.0127 0" rpy="${pi} 0.0 0.0" />
-      <limit lower="-3.14" upper="3.14" velocity="100.0" effort="0.1"/>
+      <limit lower="0" upper="0.8025" velocity="100.0" effort="0.1"/>
       <mimic joint="${prefix}robotiq_85_left_knuckle_joint" offset="0"/>
     </joint>
-    <joint name="${prefix}robotiq_85_right_inner_knuckle_joint" type="continuous">
+    <joint name="${prefix}robotiq_85_right_inner_knuckle_joint" type="revolute">
       <parent link="${prefix}robotiq_85_base_link"/>
       <child link="${prefix}robotiq_85_right_inner_knuckle_link"/>
       <axis xyz="0 0 1"/>
       <origin xyz="0.06142 -0.0127 0" rpy="0 0 0"/>
-      <limit lower="-3.14" upper="3.14" velocity="100.0" effort="0.1"/>
+      <limit lower="0" upper="0.8025" velocity="100.0" effort="0.1"/>
       <mimic joint="${prefix}robotiq_85_left_knuckle_joint" offset="0"/>
     </joint>
@@ -182,5 +182,5 @@
       </inertial>
     </link>
-    <joint name="${prefix}robotiq_85_left_finger_tip_joint" type="continuous">
+    <joint name="${prefix}robotiq_85_left_finger_tip_joint" type="revolute">
       <parent link="${prefix}robotiq_85_left_inner_knuckle_link"/>
       <child link="${prefix}robotiq_85_left_finger_tip_link"/>
@@ -190,5 +190,5 @@
       <mimic joint="${prefix}robotiq_85_left_knuckle_joint" multiplier="-1"/>
     </joint>
-    <joint name="${prefix}robotiq_85_right_finger_tip_joint" type="continuous">
+    <joint name="${prefix}robotiq_85_right_finger_tip_joint" type="revolute">
       <parent link="${prefix}robotiq_85_right_inner_knuckle_link"/>
       <child link="${prefix}robotiq_85_right_finger_tip_link"/>

Commit message: Set correct joint limits

File: src/pkg_gripper/urdf/robotiq_85_gripper.urdf.xacro (robot description, xacro)
@@ -133,5 +133,5 @@
       <axis xyz="0 0 1"/>
       <origin xyz="0.06142 0.0127 0" rpy="${pi} 0.0 0.0" />
-      <limit lower="0" upper="0.8025" velocity="100.0" effort="0.1"/>
+      <limit lower="0" upper="0.8757" velocity="100.0" effort="0.1"/>
       <mimic joint="${prefix}robotiq_85_left_knuckle_joint" offset="0"/>
     </joint>
@@ -141,5 +141,5 @@
       <axis xyz="0 0 1"/>
       <origin xyz="0.06142 -0.0127 0" rpy="0 0 0"/>
-      <limit lower="0" upper="0.8025" velocity="100.0" effort="0.1"/>
+      <limit lower="0" upper="0.8757" velocity="100.0" effort="0.1"/>
       <mimic joint="${prefix}robotiq_85_left_knuckle_joint" offset="0"/>
     </joint>
