Commit message: Add another ur5_gripper moveit config (temporary)

File: src/ur_gripper_moveit_des_config/config/gazebo_ur5_with_robotiq_2f_85.urdf (robot description, URDF)
Before this commit: robot ur5_with_robotiq_2f_85, 23 links, 22 joints
Links:
- removed link left_inner_finger
- removed link left_inner_finger_pad
- removed link left_inner_knuckle
- removed link left_outer_finger
- removed link left_outer_knuckle
- removed link right_inner_finger
- removed link right_inner_finger_pad
- removed link right_inner_knuckle
- removed link right_outer_finger
- removed link right_outer_knuckle
- removed link robotiq_arg2f_base_link
- added link robotiq_85_base_link, mass 0.636951; collision mesh filename=package://robotiq_description/meshes/collision/robotiq_85_b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; visual mesh filename=package://robotiq_description/meshes/visual/robotiq_85_base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
- added link robotiq_85_left_finger_link, mass 0.027309; collision mesh filename=package://robotiq_description/meshes/collision/robotiq_85_f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; visual mesh filename=package://robotiq_description/meshes/visual/robotiq_85_fing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
- added link robotiq_85_left_finger_tip_link, mass 0.019555; collision mesh filename=package://robotiq_description/meshes/collision/robotiq_85_f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; visual mesh filename=package://robotiq_description/meshes/visual/robotiq_85_fing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
- added link robotiq_85_left_inner_knuckle_link, mass 0.029951; collision mesh filename=package://robotiq_description/meshes/collision/robotiq_85_i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; visual mesh filename=package://robotiq_description/meshes/visual/robotiq_85_inne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
- added link robotiq_85_left_knuckle_link, mass 0.018491; collision mesh filename=package://robotiq_description/meshes/collision/robotiq_85_k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; visual mesh filename=package://robotiq_description/meshes/visual/robotiq_85_knuc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
- added link robotiq_85_right_finger_link, mass 0.027309; collision mesh filename=package://robotiq_description/meshes/collision/robotiq_85_f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; visual mesh filename=package://robotiq_description/meshes/visual/robotiq_85_fing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
- added link robotiq_85_right_finger_tip_link, mass 0.019555; collision mesh filename=package://robotiq_description/meshes/collision/robotiq_85_f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; visual mesh filename=package://robotiq_description/meshes/visual/robotiq_85_fing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
- added link robotiq_85_right_inner_knuckle_link, mass 0.029951; collision mesh filename=package://robotiq_description/meshes/collision/robotiq_85_i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; visual mesh filename=package://robotiq_description/meshes/visual/robotiq_85_inne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
- added link robotiq_85_right_knuckle_link, mass 0.018491; collision mesh filename=package://robotiq_description/meshes/collision/robotiq_85_k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; visual mesh filename=package://robotiq_description/meshes/visual/robotiq_85_knuc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
Joints:
- removed joint finger_joint
- removed joint left_inner_finger_joint
- removed joint left_inner_finger_pad_joint
- removed joint left_inner_knuckle_joint
- removed joint left_outer_finger_joint
- removed joint right_inner_finger_joint
- removed joint right_inner_finger_pad_joint
- removed joint right_inner_knuckle_joint
- removed joint right_outer_finger_joint
- removed joint right_outer_knuckle_joint
- removed joint tool_to_gripper
- added joint robotiq_85_base_joint: type fixed, parent tool0, child robotiq_85_base_link, origin xyz=0 0 0.004 rpy=0 -1.5707963267948966 3.141592653589793
- added joint robotiq_85_left_finger_joint: type fixed, parent robotiq_85_left_knuckle_link, child robotiq_85_left_finger_link, origin xyz=-0.00408552455 -0.03148604435 0.0 rpy=0 0 0
- added joint robotiq_85_left_finger_tip_joint: type continuous, parent robotiq_85_left_inner_knuckle_link, child robotiq_85_left_finger_tip_link, origin xyz=0.04303959807 -0.03759940821 0.0 rpy=0.0 0.0 0.0, axis 0 0 1, limit lower=-3.14 upper=3.14 effort=0.1 velocity=100.0, mimic joint=robotiq_85_left_knuckle_joint multiplier=-1
- added joint robotiq_85_left_inner_knuckle_joint: type continuous, parent robotiq_85_base_link, child robotiq_85_left_inner_knuckle_link, origin xyz=0.06142 0.0127 0 rpy=3.141592653589793 0.0 0.0, axis 0 0 1, limit lower=-3.14 upper=3.14 effort=0.1 velocity=100.0, mimic joint=robotiq_85_left_knuckle_joint offset=0
- added joint robotiq_85_left_knuckle_joint: type revolute, parent robotiq_85_base_link, child robotiq_85_left_knuckle_link, origin xyz=0.05490451627 0.03060114443 0.0 rpy=3.141592653589793 0.0 0.0, axis 0 0 1, limit lower=0.0 upper=0.80285 effort=1000 velocity=0.5
- added joint robotiq_85_right_finger_joint: type fixed, parent robotiq_85_right_knuckle_link, child robotiq_85_right_finger_link, origin xyz=-0.00408552455 -0.03148604435 0.0 rpy=0 0 0
- added joint robotiq_85_right_finger_tip_joint: type continuous, parent robotiq_85_right_inner_knuckle_link, child robotiq_85_right_finger_tip_link, origin xyz=0.04303959807 -0.03759940821  0.0 rpy=0.0 0.0 0.0, axis 0 0 1, limit lower=-3.14 upper=3.14 effort=0.1 velocity=100.0, mimic joint=robotiq_85_left_knuckle_joint multiplier=-1
- added joint robotiq_85_right_inner_knuckle_joint: type continuous, parent robotiq_85_base_link, child robotiq_85_right_inner_knuckle_link, origin xyz=0.06142 -0.0127 0 rpy=0 0 0, axis 0 0 1, limit lower=-3.14 upper=3.14 effort=0.1 velocity=100.0, mimic joint=robotiq_85_left_knuckle_joint offset=0
- added joint robotiq_85_right_knuckle_joint: type continuous, parent robotiq_85_base_link, child robotiq_85_right_knuckle_link, origin xyz=0.05490451627 -0.03060114443 0.0 rpy=0.0 0.0 0.0, axis 0 0 1, limit lower=-3.14 upper=3.14 effort=1000 velocity=100.0, mimic joint=robotiq_85_left_knuckle_joint

Commit message: Update gazebo

File: src/ur_gripper_moveit_des_config/config/gazebo_ur5_with_robotiq_2f_85.urdf (robot description, URDF)
Before this commit: robot ur5_with_robotiq_2f_85, 21 links, 20 joints
Joints:
- joint robotiq_85_right_knuckle_joint: mimic joint=robotiq_85_left_knuckle_joint -> (none)
