Commit message: Add virtual joint for fixing the robot to the ground (BUG of moveit)

File: src/pkg_ur_gripper_moveit/config/gazebo_ur5_with_robotiq_2f_85.urdf (robot description, URDF)
Before this commit: robot ur5_with_robotiq_2f_85, 20 links, 19 joints
Links:
- added link world
Joints:
- added joint virtual_base: type fixed, parent world, child base_link, origin xyz=0 0 0 rpy=0 0 0

Commit message: Fix urdf issues (joint limits, plugins, remove unused transmissions)

File: src/pkg_ur_gripper_moveit/config/gazebo_ur5_with_robotiq_2f_85.urdf (robot description, URDF)
Before this commit: robot ur5_with_robotiq_2f_85, 21 links, 20 joints
Joints:
- joint robotiq_85_left_inner_knuckle_joint: limit lower=0 upper=0.8025 effort=0.1 velocity=100.0 -> lower=0 upper=0.8757 effort=0.1 velocity=100.0
- joint robotiq_85_right_inner_knuckle_joint: limit lower=0 upper=0.8025 effort=0.1 velocity=100.0 -> lower=0 upper=0.8757 effort=0.1 velocity=100.0
- joint virtual_base: origin xyz=0 0 0 rpy=0 0 0 -> xyz=0 0 0.04 rpy=0 0 0

Commit message: Update load position

File: src/pkg_ur_gripper_moveit/config/gazebo_ur5_with_robotiq_2f_85.urdf (robot description, URDF)
Before this commit: robot ur5_with_robotiq_2f_85, 21 links, 20 joints
Joints:
- joint virtual_base: origin xyz=0 0 0.04 rpy=0 0 0 -> xyz=0 0 0 rpy=0 0 0
